Commit message: Adapt firmware and robot model to the confirmed drive hardware
Hardware: Arduino Mega 2560, 2x L298N, 4x JGB37-520 12V 333 RPM
gearmotors with hall encoders, 80 mm mecanum wheels.

- Firmware: L298N EN (PWM) + IN1/IN2 per wheel, per-wheel invert flag,
  quadrature A/B decoding (direction measured, not inferred from the last
  command), TICKS_PER_REV 660 (11 PPR x 2 edges x 1:30, still unverified)
- URDF + robot_params: wheel radius 0.04 m, wheel width 0.037 m

Motor pins are still copied from the previous group's robot, and the lx/ly
wheel separations are still placeholders: both must be checked on the robot.

Co-Authored-By: Claude Opus 5.5 <noreply@anthropic.com>

File: urdf/mecanum_agv.urdf.xacro (robot description, xacro)
@@ -6,6 +6,6 @@
   <xacro:property name="chassis_width" value="0.20"/>
   <xacro:property name="chassis_height" value="0.08"/>
-  <xacro:property name="wheel_radius" value="0.03"/>
-  <xacro:property name="wheel_width" value="0.03"/>
+  <xacro:property name="wheel_radius" value="0.04"/>
+  <xacro:property name="wheel_width" value="0.037"/>
   <xacro:property name="wheel_separation_x" value="0.10"/>  <!-- lx: half wheelbase -->
   <xacro:property name="wheel_separation_y" value="0.10"/>  <!-- ly: half track width -->

Commit message: Use measured chassis dimensions for kinematics, URDF and Nav2 footprint
Plate 21x21 cm, wheelbase ~17.4 cm (lx=0.087), track ~25.6 cm (ly=0.128):
18.74 cm between bracket faces + 1.6 cm gap + half of the 3.7 cm wheel per side.
Footprint 0.26 x 0.30 m covers the wheels sticking out past the plate.

Co-Authored-By: Claude Opus 5.5 <noreply@anthropic.com>

File: urdf/mecanum_agv.urdf.xacro (robot description, xacro)
@@ -1,13 +1,13 @@
 <?xml version="1.0"?>
 <robot name="mecanum_agv" xmlns:xacro="http://www.ros.org/wiki/xacro">
-  <!-- Placeholder dimensions (meters) — measure the real chassis and update these,
-       and keep wheel_radius/wheel_separation_x/y in sync with config/robot_params.yaml -->
-  <xacro:property name="chassis_length" value="0.24"/>
-  <xacro:property name="chassis_width" value="0.20"/>
+  <!-- Measured dimensions (meters) of the real chassis —
+       keep wheel_radius/wheel_separation_x/y in sync with config/robot_params.yaml -->
+  <xacro:property name="chassis_length" value="0.21"/>  <!-- measured plate: 21 x 21 cm -->
+  <xacro:property name="chassis_width" value="0.21"/>
   <xacro:property name="chassis_height" value="0.08"/>
   <xacro:property name="wheel_radius" value="0.04"/>
   <xacro:property name="wheel_width" value="0.037"/>
-  <xacro:property name="wheel_separation_x" value="0.10"/>  <!-- lx: half wheelbase -->
-  <xacro:property name="wheel_separation_y" value="0.10"/>  <!-- ly: half track width -->
+  <xacro:property name="wheel_separation_x" value="0.087"/>  <!-- lx: half wheelbase, measured just under 17.5 cm axle to axle -->
+  <xacro:property name="wheel_separation_y" value="0.128"/>  <!-- ly: half track, (18.74 cm bracket-to-bracket + 2*(1.6 gap + 3.7/2 wheel)) / 2 -->
   <xacro:property name="lidar_offset_x" value="0.0"/>
   <xacro:property name="lidar_offset_z" value="0.10"/>       <!-- height of lidar above base_link -->
